Commit message: URDF Base build Ackermann

File: src/tractor_description/urdf/robot_core.xacro (robot description, xacro)
@@ -1,24 +1,117 @@
 <?xml version="1.0"?>
 <robot xmlns:xacro="http://ros.org/wiki/xacro" name="mi_robot">
-  <xacro:include filename="colors.xacro"/>
+<!-- Desarrollo en REP 103
+Base Units
+Quantity	Unit
+length	meter
+mass	kilogram
+time	second
+current	ampere
+Derived Units
+Quantity	Unit
+angle	radian
+frequency	hertz
+force	newton
+power	watt
+voltage	volt
+temperature	celsius
+magnetism	tesla
+Chirality
+Regla de la mano derecha
+-->
+  <xacro:include filename="colors.xacro"/> <!-- Include Colors-->
+  <xacro:property name="L" value="0.148" /><!-- WheelBase -->
+  <xacro:property name="T" value="0.133" /><!-- Track -->
+  <xacro:property name="r" value="0.0325" /><!-- WheelRadius -->
+  <xacro:property name="w" value="0.025" /><!-- WheelWidth -->
+  <xacro:property name="pi" value="3.14159"/>
+  <!-- LINKS DEL ROBOT-->
   <link name="base_link">
-  </link>
-  <joint name="chassis1_joint" type="fixed">
-    <parent link="base_link"/>
-    <child link="chassis_link"/>
-    <origin xyz="0 0 0" rpy="0 0 0"/>
-  </joint>
-  <link name="chassis1_link">
     <visual>
       <geometry>
-        <box size="1.5 1.0 0.5"/>
+        <box size="${0.85*L} ${0.6*T} ${0.5*r}"/>
       </geometry>
       <material name="red"/>
-      <origin xyz="0 0 0.25" rpy="0 0 0"/>
+      <origin xyz="0 0 ${r}" rpy="0 0 0"/>
     </visual>
   </link>
-  <joint name="chassis2_joint" type="fixed">
-    <parent link="chassis1_link"/>
-    <child link="chassis2_link"/>
-    <origin xyz="0 0 0" rpy="0 0 0"/>
+  <link name="front_left_steer">
+    <visual>
+      <geometry>
+         <box size="${r*.4} ${w+0.01} ${r*.4}"/>
+      </geometry>
+      <material name="green"/>
+    </visual>
+  </link>
+  <link name="front_right_steer">
+    <visual>
+      <geometry>
+         <box size="${r*.4} ${w+0.01} ${r*.4}"/>
+      </geometry>
+      <material name="green"/>
+    </visual>
+  </link>
+  <link name="front_left_wheel">
+    <visual>
+      <geometry>
+         <cylinder radius="${r}" length="${w}"/>
+      </geometry>
+      <material name="blue"/>
+    </visual>
+  </link>
+  <link name="front_right_wheel">
+    <visual>
+      <geometry>
+         <cylinder radius="${r}" length="${w}"/>
+      </geometry>
+      <material name="blue"/>
+    </visual>
+  </link>
+  <link name="back_left_wheel">
+    <visual>
+      <geometry>
+         <cylinder radius="${r}" length="${w}"/>
+      </geometry>
+      <material name="blue"/>
+    </visual>
+  </link>
+  <link name="back_right_wheel">
+    <visual>
+      <geometry>
+         <cylinder radius="${r}" length="${w}"/>
+      </geometry>
+      <material name="blue"/>
+    </visual>
+  </link>
+  <!-- JOINTS DEL ROBOT-->
+  <joint name="joint_base_lsteer" type="fixed">
+    <parent link="base_link"/>
+    <child link="front_left_steer"/>
+    <origin xyz="${0.5*L} ${0.5*T} 0" rpy="0 0 0"/>
+  </joint>
+  <joint name="joint_base_rsteer" type="fixed">
+    <parent link="base_link"/>
+    <child link="front_right_steer"/>
+    <origin xyz="${0.5*L} ${-0.5*T} 0" rpy="0 0 0"/>
+  </joint>
+  <joint name="joint_steer_lfwheel" type="fixed">
+    <parent link="front_left_steer"/>
+    <child link="front_left_wheel"/>
+    <origin xyz="0 0 0" rpy="${pi/2} 0 0"/>
+  </joint>
+  <joint name="joint_steer_rfwheel" type="fixed">
+    <parent link="front_right_steer"/>
+    <child link="front_right_wheel"/>
+    <origin xyz="0 0 0" rpy="${pi/2} 0 0"/>
+  </joint>
+  <joint name="joint_base_lbwheel" type="fixed">
+    <parent link="base_link"/>
+    <child link="back_left_wheel"/>
+    <origin xyz="${-0.5*L} ${0.5*T} 0" rpy="${pi/2} 0 0"/>
+  </joint>
+  <joint name="joint_base_rbwheel" type="fixed">
+    <parent link="base_link"/>
+    <child link="back_right_wheel"/>
+    <origin xyz="${-0.5*L} ${-0.5*T} 0" rpy="${pi/2} 0 0"/>
+  </joint>
 </robot>

Commit message: Finished urdf visuals

File: src/tractor_description/urdf/robot_core.xacro (robot description, xacro)
@@ -35,9 +35,16 @@
       <origin xyz="0 0 ${r}" rpy="0 0 0"/>
     </visual>
+    <visual>
+      <geometry>
+        <box size="${0.425*L} ${0.6*T} ${0.5*r}"/>
+      </geometry>
+      <material name="red"/>
+      <origin xyz="${-0.2125*L} 0 ${1.5*r}" rpy="0 0 0"/>
+    </visual>
   </link>
   <link name="front_left_steer">
     <visual>
       <geometry>
-         <box size="${r*.4} ${w+0.01} ${r*.4}"/>
+         <box size="${r*.4} ${w+0.01} ${r}"/>
       </geometry>
       <material name="green"/>
@@ -47,5 +54,5 @@
     <visual>
       <geometry>
-         <box size="${r*.4} ${w+0.01} ${r*.4}"/>
+         <box size="${r*.4} ${w+0.01} ${r}"/>
       </geometry>
       <material name="green"/>
@@ -58,4 +65,11 @@
       </geometry>
       <material name="blue"/>
+      <origin xyz="0 0 0" rpy="${-pi/2} 0 0"/>
+    </visual>
+    <visual>
+      <geometry>
+          <sphere radius="0.005"/>
+      </geometry>
+      <origin xyz="0 0 ${r}" rpy="0 0 0"/>
     </visual>
   </link>
@@ -66,4 +80,11 @@
       </geometry>
       <material name="blue"/>
+      <origin xyz="0 0 0" rpy="${-pi/2} 0 0"/>
+    </visual>
+    <visual>
+      <geometry>
+          <sphere radius="0.005"/>
+      </geometry>
+      <origin xyz="0 0 ${r}" rpy="0 0 0"/>
     </visual>
   </link>
@@ -74,4 +95,11 @@
       </geometry>
       <material name="blue"/>
+      <origin xyz="0 0 0" rpy="${-pi/2} 0 0"/>
+    </visual>
+    <visual>
+      <geometry>
+          <sphere radius="0.005"/>
+      </geometry>
+      <origin xyz="0 0 ${r}" rpy="0 0 0"/>
     </visual>
   </link>
@@ -82,36 +110,51 @@
       </geometry>
       <material name="blue"/>
+      <origin xyz="0 0 0" rpy="${-pi/2} 0 0"/>
+    </visual>
+    <visual>
+      <geometry>
+          <sphere radius="0.005"/>
+      </geometry>
+      <origin xyz="0 0 ${r}" rpy="0 0 0"/>
     </visual>
   </link>
   <!-- JOINTS DEL ROBOT-->
-  <joint name="joint_base_lsteer" type="fixed">
+  <joint name="joint_base_lsteer" type="revolute">
     <parent link="base_link"/>
     <child link="front_left_steer"/>
-    <origin xyz="${0.5*L} ${0.5*T} 0" rpy="0 0 0"/>
+    <origin xyz="${0.5*L} ${0.5*T} ${r}" rpy="0 0 0"/>
+    <axis xyz="0 0 1"/>
+    <limit lower="-0.6" upper="0.6" effort="1" velocity="2.0"/>
   </joint>
-  <joint name="joint_base_rsteer" type="fixed">
+  <joint name="joint_base_rsteer" type="revolute">
     <parent link="base_link"/>
     <child link="front_right_steer"/>
-    <origin xyz="${0.5*L} ${-0.5*T} 0" rpy="0 0 0"/>
+    <origin xyz="${0.5*L} ${-0.5*T} ${r}" rpy="0 0 0"/>
+    <axis xyz="0 0 1"/>
+    <limit lower="-0.6" upper="0.6" effort="1" velocity="2.0"/>
   </joint>
-  <joint name="joint_steer_lfwheel" type="fixed">
+  <joint name="joint_steer_lfwheel" type="continuous">
     <parent link="front_left_steer"/>
     <child link="front_left_wheel"/>
-    <origin xyz="0 0 0" rpy="${pi/2} 0 0"/>
+    <origin xyz="0 0 0" rpy="0 0 0"/>
+    <axis xyz="0 1 0"/>
   </joint>
-  <joint name="joint_steer_rfwheel" type="fixed">
+  <joint name="joint_steer_rfwheel" type="continuous">
     <parent link="front_right_steer"/>
     <child link="front_right_wheel"/>
-    <origin xyz="0 0 0" rpy="${pi/2} 0 0"/>
+    <origin xyz="0 0 0" rpy="0 0 0"/>
+    <axis xyz="0 1 0"/>
   </joint>
-  <joint name="joint_base_lbwheel" type="fixed">
+  <joint name="joint_base_lbwheel" type="continuous">
     <parent link="base_link"/>
     <child link="back_left_wheel"/>
-    <origin xyz="${-0.5*L} ${0.5*T} 0" rpy="${pi/2} 0 0"/>
+    <origin xyz="${-0.5*L} ${0.5*T} ${r}" rpy="0 0 0"/>
+    <axis xyz="0 1 0"/>
   </joint>
-  <joint name="joint_base_rbwheel" type="fixed">
+  <joint name="joint_base_rbwheel" type="continuous">
     <parent link="base_link"/>
     <child link="back_right_wheel"/>
-    <origin xyz="${-0.5*L} ${-0.5*T} 0" rpy="${pi/2} 0 0"/>
+    <origin xyz="${-0.5*L} ${-0.5*T} ${r}" rpy="0 0 0"/>
+    <axis xyz="0 1 0"/>
   </joint>
 </robot>

Commit message: Sim Rdy

File: src/tractor_description/urdf/robot_core.xacro (robot description, xacro)
@@ -21,4 +21,5 @@
 -->
   <xacro:include filename="colors.xacro"/> <!-- Include Colors-->
+  <xacro:include filename="inertials.xacro"/> <!-- Include Inertia-->
   <xacro:property name="L" value="0.148" /><!-- WheelBase -->
   <xacro:property name="T" value="0.133" /><!-- Track -->
@@ -26,4 +27,7 @@
   <xacro:property name="w" value="0.025" /><!-- WheelWidth -->
   <xacro:property name="pi" value="3.14159"/>
+  <xacro:property name="m_base" value="0.40"/>   <!-- kg -->
+  <xacro:property name="m_wheel" value="0.03"/>  <!-- kg per wheel -->
+  <xacro:property name="m_steer" value="0.015"/>  <!-- kg per steer -->
   <!-- LINKS DEL ROBOT-->
   <link name="base_link">
@@ -42,4 +46,10 @@
       <origin xyz="${-0.2125*L} 0 ${1.5*r}" rpy="0 0 0"/>
     </visual>
+    <xacro:inertial_box mass="${m_base}"
+                      x="${0.80*L}"
+                      y="${0.50*T}"
+                      z="${0.40*r}"
+                      origin_xyz="0 0 ${r}"
+                      origin_rpy="0 0 0"/>
   </link>
   <link name="front_left_steer">
@@ -50,4 +60,12 @@
       <material name="green"/>
     </visual>
+    <inertial>
+      <origin xyz="0 0 0" rpy="0 0 0"/>
+      <mass value="${m_steer}"/>
+      <inertia ixx="${(m_steer/12.0)*((w+0.01)*(w+0.01) + r*r)}"
+              iyy="${(m_steer/12.0)*(1.16*r*r)}"
+              izz="${(m_steer/12.0)*(0.16*r*r + (w+0.01)*(w+0.01))}"
+              ixy="0" ixz="0" iyz="0"/>
+    </inertial>
   </link>
   <link name="front_right_steer">
@@ -58,4 +76,12 @@
       <material name="green"/>
     </visual>
+    <inertial>
+      <origin xyz="0 0 0" rpy="0 0 0"/>
+      <mass value="${m_steer}"/>
+      <inertia ixx="${(m_steer/12.0)*((w+0.01)*(w+0.01) + r*r)}"
+              iyy="${(m_steer/12.0)*(1.16*r*r)}"
+              izz="${(m_steer/12.0)*(0.16*r*r + (w+0.01)*(w+0.01))}"
+              ixy="0" ixz="0" iyz="0"/>
+    </inertial>
   </link>
   <link name="front_left_wheel">
@@ -73,4 +99,9 @@
       <origin xyz="0 0 ${r}" rpy="0 0 0"/>
     </visual>
+    <xacro:inertial_cylinder mass="${m_wheel}"
+                         radius="${r}"
+                         length="${w}"
+                         origin_xyz="0 0 0"
+                         origin_rpy="${-pi/2} 0 0"/>
   </link>
   <link name="front_right_wheel">
@@ -88,4 +119,9 @@
       <origin xyz="0 0 ${r}" rpy="0 0 0"/>
     </visual>
+    <xacro:inertial_cylinder mass="${m_wheel}"
+                         radius="${r}"
+                         length="${w}"
+                         origin_xyz="0 0 0"
+                         origin_rpy="${-pi/2} 0 0"/>
   </link>
   <link name="back_left_wheel">
@@ -103,4 +139,9 @@
       <origin xyz="0 0 ${r}" rpy="0 0 0"/>
     </visual>
+    <xacro:inertial_cylinder mass="${m_wheel}"
+                         radius="${r}"
+                         length="${w}"
+                         origin_xyz="0 0 0"
+                         origin_rpy="${-pi/2} 0 0"/>
   </link>
   <link name="back_right_wheel">
@@ -118,4 +159,9 @@
       <origin xyz="0 0 ${r}" rpy="0 0 0"/>
     </visual>
+    <xacro:inertial_cylinder mass="${m_wheel}"
+                         radius="${r}"
+                         length="${w}"
+                         origin_xyz="0 0 0"
+                         origin_rpy="${-pi/2} 0 0"/>
   </link>
   <!-- JOINTS DEL ROBOT-->
@@ -126,4 +172,5 @@
     <axis xyz="0 0 1"/>
     <limit lower="-0.6" upper="0.6" effort="1" velocity="2.0"/>
+    <dynamics damping="0.1" friction="0.02"/>
   </joint>
   <joint name="joint_base_rsteer" type="revolute">
@@ -133,4 +180,5 @@
     <axis xyz="0 0 1"/>
     <limit lower="-0.6" upper="0.6" effort="1" velocity="2.0"/>
+    <dynamics damping="0.1" friction="0.02"/>
   </joint>
   <joint name="joint_steer_lfwheel" type="continuous">

Commit message: Fix inertial URDF

File: src/tractor_description/urdf/robot_core.xacro (robot description, xacro)
@@ -31,4 +31,5 @@
   <xacro:property name="m_steer" value="0.015"/>  <!-- kg per steer -->
   <!-- LINKS DEL ROBOT-->
+  <link name="base_footprint"/>
   <link name="base_link">
     <visual>
@@ -166,4 +167,11 @@
   </link>
   <!-- JOINTS DEL ROBOT-->
+  <!-- 2) Fija base_footprint -> base_link -->
+  <joint name="base_footprint_to_base_link" type="fixed">
+    <parent link="base_footprint"/>
+    <child link="base_link"/>
+    <!-- Si tu base_link ya está a z=0 en el suelo, deja en 0 -->
+    <origin xyz="0 0 0" rpy="0 0 0"/>
+  </joint>
   <joint name="joint_base_lsteer" type="revolute">
     <parent link="base_link"/>
